Commit message: mimic

File: draco/draco.urdf (robot description, URDF)
Before this commit: robot draco, 40 links, 39 joints
Links:
- link l_wrist_pitch_link: geometry 
- link r_wrist_pitch_link: geometry 
Joints:
- joint l_knee_fe_jd: mimic (none) -> joint=l_knee_fe_jp multiplier=1.0 offset=0.0
- joint r_knee_fe_jd: mimic (none) -> joint=r_knee_fe_jp multiplier=1.0 offset=0.0
