Commit message: working bbot

File: bumpybot/bumpybot.urdf (robot description, URDF)
Before this commit: robot bumpybot, 4 links, 3 joints
Links:
- removed link dummy_x_link
- removed link dummy_y_link
- removed link dummy_yaw_link
- added link dummy_prismatic_x_link, mass 1e-9
- added link dummy_prismatic_y_link, mass 1e-9
- added link dummy_revolute_yaw_link, mass 20; collision cylinder length=0.6318758 radius=0.3048; visual mesh filename=package://meshes/bumpybot_exterior.stl scale=0.0009 0.0009 0.0009
Joints:
- removed joint dummy_x_joint
- removed joint dummy_y_joint
- removed joint dummy_yaw_joint
- added joint dummy_prismatic_x_joint: type prismatic, parent base_link, child dummy_prismatic_x_link, origin xyz=0 0 0, axis 1 0 0, limit lower=-20 upper=20 effort=1000.0 velocity=10
- added joint dummy_prismatic_y_joint: type prismatic, parent dummy_prismatic_x_link, child dummy_prismatic_y_link, origin xyz=0 0 0, axis 0 1 0, limit lower=-20 upper=20 effort=1000.0 velocity=10
- added joint dummy_revolute_yaw_joint: type revolute, parent dummy_prismatic_y_link, child dummy_revolute_yaw_link, origin xyz=0 0 0, axis 0 0 1, limit lower=-100 upper=100 effort=1000.0 velocity=10

Commit message: bumpybot testing objects

File: bumpybot/bumpybot.urdf (robot description, URDF)
Before this commit: robot bumpybot, 4 links, 3 joints
Links:
- removed link base_link
- added link base, mass 1e-9; visual cylinder length=0.4 radius=0.1
- link dummy_prismatic_x_link: geometry visual cylinder length=0.4 radius=0.1
- link dummy_prismatic_y_link: geometry visual cylinder length=0.4 radius=0.1
- link dummy_revolute_yaw_link: geometry visual mesh filename=package://meshes/bumpybot_full.stl scale=0.0015 0.0015 0.0015
Joints:
- joint dummy_prismatic_x_joint: parent base_link -> base
- joint dummy_revolute_yaw_joint: axis 0 0 1 -> 0 0 0

Commit message: fixed virtual floating links

File: bumpybot/bumpybot.urdf (robot description, URDF)
Before this commit: robot bumpybot, 4 links, 3 joints
Links:
- removed link dummy_revolute_yaw_link
- added link robot_link, mass 20; collision cylinder length=0.685 radius=0.3048; visual mesh filename=package://meshes/bumpybot_full.stl scale=0.0015 0.0015 0.0015
- link base: mass 1e-9 -> 1e9; geometry 
- link dummy_prismatic_x_link: geometry 
- link dummy_prismatic_y_link: geometry 
Joints:
- joint dummy_prismatic_x_joint: limit lower=-20 upper=20 effort=1000.0 velocity=10 -> lower=-100 upper=100 effort=1000.0 velocity=10; origin xyz=0 0 0 -> xyz=0 0 0 rpy=0 0 0
- joint dummy_prismatic_y_joint: limit lower=-20 upper=20 effort=1000.0 velocity=10 -> lower=-100 upper=100 effort=1000.0 velocity=10; origin xyz=0 0 0 -> xyz=0 0 0 rpy=0 0 0
- joint dummy_revolute_yaw_joint: axis 0 0 0 -> 0 0 1; child dummy_revolute_yaw_link -> robot_link; limit lower=-100 upper=100 effort=1000.0 velocity=10 -> lower=-1e9 upper=1e9 effort=1000.0 velocity=10; origin xyz=0 0 0 -> xyz=0 0 0 rpy=0 0 0

Commit message: expand joint lims for bumpybot

File: bumpybot/bumpybot.urdf (robot description, URDF)
Before this commit: robot bumpybot, 4 links, 3 joints
Joints:
- joint dummy_prismatic_x_joint: limit lower=-100 upper=100 effort=1000.0 velocity=10 -> lower=-1e9 upper=1e9 effort=1000.0 velocity=10
- joint dummy_prismatic_y_joint: limit lower=-100 upper=100 effort=1000.0 velocity=10 -> lower=-1e9 upper=1e9 effort=1000.0 velocity=10
