Commit message: bumpybot collision box

File: bumpybot/bumpybot_simple.urdf (robot description, URDF)
Before this commit: robot so2, 4 links, 3 joints
Links:
- link base: geometry collision cylinder length=0.4 radius=0.36; visual mesh filename=meshes/bumpybot_full.stl scale=0.001 0.001 0.001

Commit message: better bbot capsule collision

File: bumpybot/bumpybot_simple.urdf (robot description, URDF)
Before this commit: robot se2, 4 links, 3 joints
Links:
- link base: geometry collision cylinder length=0.1 radius=0.36; visual mesh filename=meshes/bumpybot_full.stl scale=0.001 0.001 0.001
