Commit message: plato/panda collision fix and simplified plato

File: plato/panda_old.urdf (robot description, URDF)
Before this commit: robot panda, 9 links, 8 joints
Links:
- link panda_link0: mass 0.629769 -> None
- link panda_link1: mass 4.970684 -> None
- link panda_link2: mass 0.646926 -> None
- link panda_link3: mass 3.228604 -> None; geometry collision cylinder length=0.15 radius=0.09; collision sphere radius=0.09
- link panda_link4: mass 3.587895 -> None
- link panda_link5: mass 1.225946 -> None
- link panda_link6: mass 1.666555 -> None
- link panda_link7: mass 0.735522 -> None; geometry collision cylinder length=0.14 radius=0.07; collision sphere radius=0.07
- link panda_link8: mass 0.73 -> None
