Commit message: Fixed the frame and joint orientations for plato

File: plato/panda_plato.urdf (robot description, URDF)
Before this commit: robot panda, 20 links, 19 joints
Links:
- added link plato_ee, mass 1e-8
Joints:
- removed joint plato_finger0_ee
- removed joint plato_finger1_ee
- removed joint plato_finger2_ee
- added joint panda_ee_joint: type fixed, parent plato_base, child plato_ee, origin xyz=0.12 0 -0.05 rpy=0 0 0
- added joint plato_finger0_ee_joint: type fixed, parent plato_finger0_link2, child plato_finger0_ee, origin xyz=0.063094028360469539551 0.0092379839030397731259 -0.0025000000000000160982 rpy=-3.1415926535897926719 1.0178922239597187368e-17 -0.016022148110467510085, axis 0 0 0
- added joint plato_finger1_ee_joint: type fixed, parent plato_finger1_link2, child plato_finger1_ee, origin xyz=0.063094028360469539551 -0.0092379839030397731259 -0.0025000000000000230371 rpy=1.5707963267948958919 1.0178915901030053653e-17 0.016022148110467458043, axis 0 0 0
- added joint plato_finger2_ee_joint: type fixed, parent plato_finger2_link2, child plato_finger2_ee, origin xyz=0.063094028360469511796 -0.009237983903039766187 -0.0024999999999999814038 rpy=1.5707963267948970021 -1.017893310654182657e-17 0.016022148110467461513, axis 0 0 0
- joint panda_joint6: limit lower=-0.0175 upper=3.7525 effort=12 velocity=2.6100 -> lower=-3.0925 upper=0.6425 effort=12 velocity=2.6100; origin xyz=0 0 0 rpy=1.5707963267948966 0 0 -> xyz=0 0 0 rpy=1.5707963267948966 -3.14 0

Commit message: fixed finger ee joint & deleted old urdfs

File: plato/panda_plato.urdf (robot description, URDF)
Before this commit: robot panda, 21 links, 20 joints
Joints:
- removed joint panda_ee_joint
- added joint plato_ee_joint: type fixed, parent plato_base, child plato_ee, origin xyz=0.2 0 -0.07 rpy=0 0 0
