Commit message: plato virtual arm

File: plato/virtual_plato.urdf (robot description, URDF)
Before this commit: robot platov2, 17 links, 16 joints
Links:
- added link virtual_link_pitch, mass 1e-9
- added link virtual_link_yaw, mass 1e-9
Joints:
- removed joint virtual_joint_plato_pitch
- added joint virtual_joint_pitch: type revolute, parent virtual_link_z, child virtual_link_pitch, origin xyz=0 0 0 rpy=0 0 0, axis 0 1 0, limit lower=-1.57 upper=1.57 effort=1000.0 velocity=10
- added joint virtual_joint_roll: type revolute, parent virtual_link_yaw, child plato_base, origin xyz=0 0 0 rpy=0 0 0, axis 1 0 0, limit lower=-1.57 upper=1.57 effort=1000.0 velocity=10
- added joint virtual_joint_yaw: type revolute, parent virtual_link_pitch, child virtual_link_yaw, origin xyz=0 0 0 rpy=0 0 0, axis 0 0 1, limit lower=-1.57 upper=1.57 effort=1000.0 velocity=10
- joint plato_ee_joint: origin xyz=0.2 0 -0.07 rpy=0 0 0 -> xyz=0.175 0 -0.07 rpy=0 0 0

Commit message: redid the collision mesh

File: plato/virtual_plato.urdf (robot description, URDF)
Before this commit: robot platov2, 19 links, 18 joints
Links:
- link plato_base: geometry collision box size=0.11 0.06 0.075; visual mesh filename=package://meshes/plato/plato_base_visual.stl
- link plato_finger0_actuator: geometry collision box size=0.07 0.025 0.04; visual mesh filename=package://meshes/plato/plato_finger0_actuator_visual.stl
