Commit message: husky cylinder collision meshes

File: husky/husky.urdf (robot description, URDF)
Before this commit: robot husky, 10 links, 9 joints
Links:
- link front_left_wheel_link: geometry collision cylinder length=0.1143 radius=0.1651; visual mesh filename=meshes/wheel.dae
- link front_right_wheel_link: geometry collision cylinder length=0.1143 radius=0.1651; visual mesh filename=meshes/wheel.dae
- link rear_left_wheel_link: geometry collision cylinder length=0.1143 radius=0.1651; visual mesh filename=meshes/wheel.dae
- link rear_right_wheel_link: geometry collision cylinder length=0.1143 radius=0.1651; visual mesh filename=meshes/wheel.dae
Joints:
- joint rear_left_wheel: mimic (none) -> joint=front_left_wheel multiplier=1.0 offset=0.0
- joint rear_right_wheel: mimic (none) -> joint=front_right_wheel multiplier=1.0 offset=0.0
