Commit message: g1 and updated t1

File: g1/g1_29dof_lock_waist_rev_1_0.urdf (robot description, URDF)
Before this commit: robot g1_29dof_lock_waist_rev_1_0, 39 links, 38 joints
Links:
- link head_link: geometry visual mesh filename=meshes/head_link.STL
- link left_elbow_link: geometry visual mesh filename=meshes/left_elbow_link.STL
- link left_hip_pitch_link: geometry visual mesh filename=meshes/left_hip_pitch_link.STL
- link left_hip_roll_link: geometry visual mesh filename=meshes/left_hip_roll_link.STL
- link left_hip_yaw_link: geometry visual mesh filename=meshes/left_hip_yaw_link.STL
- link left_knee_link: geometry collision cylinder length=0.2 radius=0.025; visual mesh filename=meshes/left_knee_link.STL
- link left_shoulder_pitch_link: geometry visual mesh filename=meshes/left_shoulder_pitch_link.STL
- link left_shoulder_roll_link: geometry visual mesh filename=meshes/left_shoulder_roll_link.STL
- link left_wrist_roll_link: geometry visual mesh filename=meshes/left_wrist_roll_link.STL
- link left_wrist_yaw_link: geometry visual mesh filename=meshes/left_wrist_yaw_link.STL
- link right_elbow_link: geometry visual mesh filename=meshes/right_elbow_link.STL
- link right_hip_pitch_link: geometry visual mesh filename=meshes/right_hip_pitch_link.STL
- link right_hip_roll_link: geometry visual mesh filename=meshes/right_hip_roll_link.STL
- link right_hip_yaw_link: geometry visual mesh filename=meshes/right_hip_yaw_link.STL
- link right_knee_link: geometry collision cylinder length=0.2 radius=0.025; visual mesh filename=meshes/right_knee_link.STL
- link right_shoulder_pitch_link: geometry visual mesh filename=meshes/right_shoulder_pitch_link.STL
- link right_shoulder_roll_link: geometry visual mesh filename=meshes/right_shoulder_roll_link.STL
- link right_wrist_roll_link: geometry visual mesh filename=meshes/right_wrist_roll_link.STL
- link right_wrist_yaw_link: geometry visual mesh filename=meshes/right_wrist_yaw_link.STL

File: t1/t1.urdf (robot description, URDF)
Before this commit: robot T1, 24 links, 23 joints
Links:
- link al3: geometry collision cylinder length=0.15 radius=0.03; visual mesh filename=meshes/AL3.STL
- link al4: geometry collision cylinder length=0.175 radius=0.03; visual mesh filename=meshes/left_hand_link.STL
- link ar3: geometry collision cylinder length=0.15 radius=0.03; visual mesh filename=meshes/AR3.STL
- link ar4: geometry collision cylinder length=0.175 radius=0.03; visual mesh filename=meshes/right_hand_link.STL
- link h2: geometry collision sphere radius=0.08; visual mesh filename=meshes/H2.STL
- link ll3: geometry collision cylinder length=0.16 radius=0.05; visual mesh filename=meshes/Hip_Yaw_Left.STL
- link ll4: geometry collision cylinder length=0.15 radius=0.05; visual mesh filename=meshes/Shank_Left.STL
- link lr3: geometry collision cylinder length=0.16 radius=0.05; visual mesh filename=meshes/Hip_Yaw_Right.STL
- link lr4: geometry collision cylinder length=0.15 radius=0.05; visual mesh filename=meshes/Shank_Right.STL
- link trunk: geometry collision box size=0.15 0.2 0.3; visual mesh filename=meshes/Trunk.STL
Joints:
- joint joint_al1: limit lower=-3.2812189937493397 upper=1.186823891356144 effort=100 velocity=50 -> lower=-3.31 upper=1.22 effort=18 velocity=18.84
- joint joint_al2: limit lower=-1.6406094968746698 upper=1.53588974175501 effort=100 velocity=50 -> lower=-1.74 upper=1.57 effort=18 velocity=18.84; origin xyz=0 0.047 0 rpy=-1.45 0 0 -> xyz=0 0.047 0 rpy=0 0 0
- joint joint_al3: limit lower=-2.0943951023931953 upper=0.03490658503988659 effort=100 velocity=50 -> lower=-2.27 upper=2.27 effort=18 velocity=18.84
- joint joint_al4: limit lower=-2.234021442552742 upper=2.234021442552742 effort=100 velocity=50 -> lower=-2.44 upper=0 effort=18 velocity=18.84
- joint joint_ar1: limit lower=-3.2812189937493397 upper=1.186823891356144 effort=100 velocity=50 -> lower=-3.31 upper=1.22 effort=18 velocity=18.84
- joint joint_ar2: limit lower=-1.53588974175501 upper=1.6406094968746698 effort=100 velocity=50 -> lower=-1.57 upper=1.74 effort=18 velocity=18.84; origin xyz=0 -0.047 0 rpy=1.45 0 0 -> xyz=0 -0.047 0 rpy=0 0 0
- joint joint_ar3: limit lower=-0.03490658503988659 upper=2.0943951023931953 effort=100 velocity=50 -> lower=-2.27 upper=2.27 effort=18 velocity=18.84
- joint joint_ar4: limit lower=-2.234021442552742 upper=2.234021442552742 effort=100 velocity=50 -> lower=0 upper=2.44 effort=18 velocity=18.84
- joint joint_h1: limit lower=-1.0122909661567112 upper=1.0122909661567112 effort=100 velocity=50 -> lower=-1.57 upper=1.57 effort=7 velocity=12.56
- joint joint_h2: limit lower=-0.3141592653589793 upper=0.8203047484373349 effort=100 velocity=50 -> lower=-0.35 upper=1.22 effort=7 velocity=12.56
- joint joint_ll1: limit lower=-2.0594885173533086 upper=2.0594885173533086 effort=100 velocity=50 -> lower=-1.8 upper=1.57 effort=45 velocity=12.5
- joint joint_ll2: limit lower=-0.3665191429188092 upper=1.53588974175501 effort=100 velocity=50 -> lower=-0.2 upper=1.57 effort=30 velocity=10.9
- joint joint_ll3: limit lower=-1.0122909661567112 upper=1.0122909661567112 effort=100 velocity=50 -> lower=-1 upper=1 effort=30 velocity=10.9
- joint joint_ll4: limit lower=-0.19198621771937624 upper=2.1467549799530254 effort=100 velocity=50 -> lower=0 upper=2.34 effort=60 velocity=11.7
- joint joint_ll5: limit lower=-0.40142572795869574 upper=0.8552113334772213 effort=100 velocity=50 -> lower=-0.87 upper=0.35 effort=20 velocity=18.8
- joint joint_ll6: limit lower=-0.41887902047863906 upper=0.7853981633974483 effort=100 velocity=50 -> lower=-0.44 upper=0.44 effort=15 velocity=12.4
- joint joint_lr1: limit lower=-2.0594885173533086 upper=2.0594885173533086 effort=100 velocity=50 -> lower=-1.8 upper=1.57 effort=45 velocity=12.5
- joint joint_lr2: limit lower=-1.53588974175501 upper=0.3665191429188092 effort=100 velocity=50 -> lower=-1.57 upper=0.2 effort=30 velocity=10.9
- joint joint_lr3: limit lower=-1.0122909661567112 upper=1.0122909661567112 effort=100 velocity=50 -> lower=-1 upper=1 effort=30 velocity=10.9
- joint joint_lr4: limit lower=-0.19198621771937624 upper=2.1467549799530254 effort=100 velocity=50 -> lower=0 upper=2.34 effort=60 velocity=11.7
- joint joint_lr5: limit lower=-0.40142572795869574 upper=0.8552113334772213 effort=100 velocity=50 -> lower=-0.87 upper=0.35 effort=20 velocity=18.8
- joint joint_lr6: limit lower=-0.41887902047863906 upper=0.7853981633974483 effort=100 velocity=50 -> lower=-0.44 upper=0.44 effort=15 velocity=12.4
- joint joint_waist: limit lower=-1.0122909661567112 upper=1.0122909661567112 effort=100 velocity=50 -> lower=-1.57 upper=1.57 effort=30 velocity=10.88
