Commit message: Isolated fingernail link

File: plato/robot/panda_plato.urdf (robot description, URDF)
Before this commit: robot panda, 18 links, 17 joints
Links:
- added link plato_finger0_linknail, mass 0.000663; collision mesh filename=package://meshes/plato/plato_finger0_nail.stl; visual mesh filename=package://meshes/plato/plato_finger0_nail.stl
- added link plato_finger1_linknail, mass 0.000663; collision mesh filename=package://meshes/plato/plato_finger1_nail.stl; visual mesh filename=package://meshes/plato/plato_finger1_nail.stl
- added link plato_finger2_linknail, mass 0.000663; collision mesh filename=package://meshes/plato/plato_finger2_nail.stl; visual mesh filename=package://meshes/plato/plato_finger2_nail.stl
- link plato_finger0_link2: mass 0.0476864 -> 0.0470234; geometry collision mesh filename=package://meshes/plato/plato_finger0_link2.stl; visual mesh filename=package://meshes/plato/plato_finger0_link2.stl
- link plato_finger1_link2: mass 0.0476874 -> 0.0470234; geometry collision mesh filename=package://meshes/plato/plato_finger1_link2.stl; visual mesh filename=package://meshes/plato/plato_finger1_link2.stl
- link plato_finger2_link2: mass 0.0476864 -> 0.0470234; geometry collision mesh filename=package://meshes/plato/plato_finger2_link2.stl; visual mesh filename=package://meshes/plato/plato_finger2_link2.stl
Joints:
- added joint plato_finger0_jointnail: type fixed, parent plato_finger0_link2, child plato_finger0_linknail, origin xyz=0 0 0 rpy=0 0 0
- added joint plato_finger1_jointnail: type fixed, parent plato_finger1_link2, child plato_finger1_linknail, origin xyz=0 0 0 rpy=0 0 0
- added joint plato_finger2_jointnail: type fixed, parent plato_finger2_link2, child plato_finger2_linknail, origin xyz=0 0 0 rpy=0 0 0

Commit message: misc changes

File: plato/robot/panda_plato.urdf (robot description, URDF)
Before this commit: robot panda, 21 links, 20 joints
Joints:
- joint plato_finger0_joint1: origin xyz=-0.0255 -0.007 -0.024 rpy=1.5708 -1.6883e-17 -3.14159 -> xyz=-0.0255 -0.007 -0.024 rpy=1.5708 0 -3.14159
- joint plato_finger0_joint2: origin xyz=0.06 0 -0.005 rpy=3.14159 -3.41605e-23 -4.23275e-16 -> xyz=0.06 0 -0.005 rpy=3.14159 0 0
- joint plato_finger0_jointnail: origin xyz=0 0 0 rpy=0 0 0 -> xyz=0.01 -0.0005 0 rpy=0 0 0
- joint plato_finger1_jointnail: origin xyz=0 0 0 rpy=0 0 0 -> xyz=0.01 0.0005 0 rpy=0 0 0
- joint plato_finger2_jointnail: origin xyz=0 0 0 rpy=0 0 0 -> xyz=0.01 0.0005 0 rpy=0 0 0

Commit message: simplified urdf collision

File: plato/robot/panda_plato.urdf (robot description, URDF)
Before this commit: robot panda, 21 links, 20 joints
Links:
- link panda_link0: geometry collision cylinder length=0.03 radius=0.09; visual mesh filename=package://meshes/visual/link0.dae
- link panda_link1: geometry collision cylinder length=0.2830 radius=0.09; visual mesh filename=package://meshes/visual/link1.dae
- link panda_link2: geometry collision cylinder length=0.26 radius=0.09; visual mesh filename=package://meshes/visual/link2.dae
- link panda_link4: geometry collision cylinder length=0.22 radius=0.09; visual mesh filename=package://meshes/visual/link4.dae
- link panda_link5: geometry collision cylinder length=0.1 radius=0.09; collision cylinder length=0.14 radius=0.055
- link panda_link6: geometry collision cylinder length=0.20 radius=0.08; visual mesh filename=package://meshes/visual/link6.dae
- link plato_base: geometry collision box size=0.11 0.06 0.075; collision cylinder length=0.04 radius=0.025

Commit message: added plato motor test bed

File: plato/robot/panda_plato.urdf (robot description, URDF)
Before this commit: robot panda, 21 links, 20 joints
Joints:
- joint plato_ee_joint: origin xyz=0.175 0 -0.07 rpy=0 0 0 -> xyz=0.175 0.04 -0.07 rpy=0 0 0
- joint plato_finger0_jointnail: origin xyz=0.01 -0.0005 0 rpy=0 0 0 -> xyz=0 -0.0005 0 rpy=0 0 0
- joint plato_finger1_jointnail: origin xyz=0.01 0.0005 0 rpy=0 0 0 -> xyz=0 0.0005 0 rpy=0 0 0
- joint plato_finger2_jointnail: origin xyz=0.01 0.0005 0 rpy=0 0 0 -> xyz=0 0.0005 0 rpy=0 0 0
