Commit message: Added Plato to Optimo urdf

File: plato/robot_optimo/optimo.urdf (robot description, URDF)
Before this commit: robot optimo, 9 links, 8 joints
Links:
- link optimo_link0: geometry collision mesh filename=package://meshes/optimo/col0.stl; visual mesh filename=package://meshes/optimo/J0_clean.stl
- link optimo_link1: geometry collision mesh filename=package://meshes/optimo/col1.stl; visual mesh filename=package://meshes/optimo/J1_clean.stl
- link optimo_link2: geometry collision mesh filename=package://meshes/optimo/col2.stl; visual mesh filename=package://meshes/optimo/J2_clean.stl
- link optimo_link3: geometry collision mesh filename=package://meshes/optimo/col3.stl; visual mesh filename=package://meshes/optimo/J3_clean.stl
- link optimo_link4: geometry collision mesh filename=package://meshes/optimo/col4.stl; visual mesh filename=package://meshes/optimo/J4_clean.stl
- link optimo_link5: geometry collision mesh filename=package://meshes/optimo/col5.stl; visual mesh filename=package://meshes/optimo/J5_clean.stl
- link optimo_link6: geometry collision mesh filename=package://meshes/optimo/col6.stl; visual mesh filename=package://meshes/optimo/J6_clean.stl
- link optimo_link7: geometry collision mesh filename=package://meshes/optimo/col7.stl; visual mesh filename=package://meshes/optimo/J7_clean.stl
