Commit message: Isolated fingernail and fingerpad on Plato

File: plato/robot_optimo/optimo_plato.urdf (robot description, URDF)
Before this commit: robot optimo, 19 links, 18 joints
Links:
- added link plato_finger1_nail, mass 1e-8; collision mesh filename=package://meshes/plato/finger_nail.stl; visual mesh filename=package://meshes/plato/finger_nail.stl
- added link plato_finger1_pad, mass 1e-8; collision mesh filename=package://meshes/plato/gel_2x4_silicone.stl; visual mesh filename=package://meshes/plato/gel_2x4_silicone.stl
- added link plato_finger2_nail, mass 1e-8; collision mesh filename=package://meshes/plato/finger_nail.stl; visual mesh filename=package://meshes/plato/finger_nail.stl
- added link plato_finger2_pad, mass 1e-8; collision mesh filename=package://meshes/plato/gel_2x4_silicone.stl; visual mesh filename=package://meshes/plato/gel_2x4_silicone.stl
- added link plato_finger3_nail, mass 1e-8; collision mesh filename=package://meshes/plato/finger_nail.stl; visual mesh filename=package://meshes/plato/finger_nail.stl
- added link plato_finger3_pad, mass 1e-8; collision mesh filename=package://meshes/plato/gel_2x4_silicone.stl; visual mesh filename=package://meshes/plato/gel_2x4_silicone.stl
- link plato_finger1_link2: geometry collision mesh filename=package://meshes/plato/plato_finger1_link2.stl; visual mesh filename=package://meshes/plato/plato_finger1_link2.stl
- link plato_finger2_link2: geometry collision mesh filename=package://meshes/plato/plato_finger2_link2.stl; visual mesh filename=package://meshes/plato/plato_finger2_link2.stl
- link plato_finger3_link2: geometry collision mesh filename=package://meshes/plato/plato_finger3_link2.stl; visual mesh filename=package://meshes/plato/plato_finger3_link2.stl
Joints:
- added joint plato_finger1_jointnail: type fixed, parent plato_finger1_link2, child plato_finger1_nail, origin xyz=0 -0.0005 0 rpy=0 0 0
- added joint plato_finger1_pad: type fixed, parent plato_finger1_link2, child plato_finger1_pad, origin xyz=0 -0.0005 0 rpy=0 0 0
- added joint plato_finger2_jointnail: type fixed, parent plato_finger2_link2, child plato_finger2_nail, origin xyz=0 0 0 rpy=0 0 0
- added joint plato_finger2_pad: type fixed, parent plato_finger2_link2, child plato_finger2_pad, origin xyz=0 0 0 rpy=0 0 0
- added joint plato_finger3_jointnail: type fixed, parent plato_finger3_link2, child plato_finger3_nail, origin xyz=0 0 0 rpy=0 0 0
- added joint plato_finger3_pad: type fixed, parent plato_finger3_link2, child plato_finger3_pad, origin xyz=0 0 0 rpy=0 0 0
- joint plato_ee_joint: origin xyz=0.0 -0.175 -0.07 rpy=0 0 0 -> xyz=0.0 -0.175 -0.07 rpy=0 0 -1.5708
