Commit message: created spacecraft robot usd

File: spacecraft/spacecraft.urdf (robot description, URDF)
Before this commit: robot Chaser, 4 links, 3 joints
Links:
- removed link Fixture
- removed link Left_Panel
- removed link Right_Panel
- removed link Spacecraft
- added link base_link, mass 0.001
- added link body, mass 100; collision box size=1.25 1.5 2; visual box size=1.25 1.5 2
- added link fixture, mass 1; collision sphere radius=0.1; visual sphere radius=0.1
- added link left_panel, mass 20; collision box size=0.25 3 1.5; visual box size=0.25 3 1.5
- added link right_panel, mass 20; collision box size=0.25 3 1.5; visual box size=0.25 3 1.5
Joints:
- removed joint Spacecraft_Fixture
- removed joint Spacecraft_Left_Panel
- removed joint Spacecraft_Right_Panel
- added joint base_to_body: type fixed, parent base_link, child body, origin xyz=0 0 0 rpy=0 0 0
- added joint body_fixture: type fixed, parent body, child fixture, origin xyz=0 0 1 rpy=0 0 0
- added joint body_left_panel: type fixed, parent body, child left_panel, origin xyz=0 -0.75 0 rpy=0 0 0
- added joint body_right_panel: type fixed, parent body, child right_panel, origin xyz=0 0.75 0 rpy=0 0 0
