Commit message: turn off most collisions and use ut colors

File: so101/so101.urdf (robot description, URDF)
Before this commit: robot so101, 8 links, 7 joints
Links:
- link base_link: geometry visual mesh filename=meshes/base_motor_holder_so101_v1.stl; visual mesh filename=meshes/base_so101_v2.stl
- link gripper_link: geometry collision mesh filename=meshes/wrist_roll_follower_so101_v1.stl; visual mesh filename=meshes/sts3215_03a_v1.stl
- link lower_arm_link: geometry visual mesh filename=meshes/motor_holder_so101_wrist_v1.stl; visual mesh filename=meshes/sts3215_03a_v1.stl
- link shoulder_link: geometry collision box size=0.1 0.1 0.05; visual mesh filename=meshes/motor_holder_so101_base_v1.stl
- link upper_arm_link: geometry visual mesh filename=meshes/sts3215_03a_v1.stl; visual mesh filename=meshes/upper_arm_so101_v1.stl
- link wrist_link: geometry visual mesh filename=meshes/sts3215_03a_no_horn_v1.stl; visual mesh filename=meshes/wrist_roll_pitch_so101_v2.stl

Commit message: update so101 collisions

File: so101/so101.urdf (robot description, URDF)
Before this commit: robot so101, 8 links, 7 joints
Links:
- removed link gripper_frame_link
Joints:
- removed joint gripper_frame_joint
